File: hardware/D1 Breakout - LCD TH Dupont.sch (EAGLE design)
At the start: 8 parts, among them J1 RJ11-4L-B

Commit message: Change level shifter to most recent version
- move from https://www.sparkfun.com/products/retired/8745
  to https://www.sparkfun.com/products/12009
Parts:
- U$3: value LOGIC_LEVEL_CONVERTER -> SPARKFUN-BOARDS_LOGIC_LEVEL_CONVERTER; device SparkFun-Boards:LOGIC_LEVEL_CONVERTER -> D1 Breakout - LCD TH Dupont:SPARKFUN-BOARDS_LOGIC_LEVEL_CONVERTER
Connections:
- net N$1: now also U$3.LV1; no longer U$3.LV_TXI_1
- net N$2: now also U$3.LV2; no longer U$3.LV_RXO_1
- net N$4: now also U$3.HV1; no longer U$3.HV_TXO_1
- net N$5: now also U$3.HV2; no longer U$3.HV_RXI_1
Changed lines of the file:
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@@
 <?xml version="1.0" encoding="utf-8"?>
 <!DOCTYPE eagle SYSTEM "eagle.dtd">
-<eagle version="7.3.0">
+<eagle version="7.7.0">
 <drawing>
 <settings>
@@
 <layer number="59" name="tCarbon" color="7" fill="1" visible="no" active="no"/>
 <layer number="60" name="bCarbon" color="7" fill="1" visible="no" active="no"/>
+<layer number="88" name="SimResults" color="9" fill="1" visible="yes" active="yes"/>
+<layer number="89" name="SimProbes" color="9" fill="1" visible="yes" active="yes"/>
 <layer number="90" name="Modules" color="5" fill="1" visible="yes" active="yes"/>
 <layer number="91" name="Nets" color="2" fill="1" visible="yes" active="yes"/>
@@
 <part name="J1" library="con-tycoelectronics" deviceset="RJ11" device="" technology="-4L-B"/>
 <part name="R1" library="rcl" deviceset="R-US_" device="0207/5V" value="10k"/>
-<part name="U$3" library="SparkFun-Boards" deviceset="LOGIC_LEVEL_CONVERTER" device=""/>
+<part name="U$3" library="D1 Breakout - LCD TH Dupont" deviceset="SPARKFUN-BOARDS_LOGIC_LEVEL_CONVERTER" device=""/>
 <part name="BZR" library="pinhead" deviceset="PINHD-1X2" device=""/>
 <part name="RELAY" library="con-lstb" deviceset="MA04-1" device=""/>
@@
 </plain>
 <instances>
-<instance part="U$1" gate="G$1" x="48.26" y="50.8"/>
-<instance part="X" gate="-1" x="63.5" y="33.02" rot="R90"/>
-<instance part="X" gate="-2" x="68.58" y="33.02" rot="R90"/>
-<instance part="J1" gate="G$1" x="22.86" y="40.64" rot="R180"/>
-<instance part="R1" gate="G$1" x="33.02" y="35.56" rot="R90"/>
-<instance part="U$3" gate="G$1" x="116.84" y="43.18"/>
-<instance part="BZR" gate="G$1" x="48.26" y="83.82"/>
-<instance part="RELAY" gate="1" x="15.24" y="73.66"/>
-<instance part="LCD" gate="1" x="116.84" y="25.4" rot="R180"/>
+<instance part="U$1" gate="G$1" x="48.26" y="50.8" smashed="yes">
+<attribute name="NAME" x="48.26" y="74.422" size="1.27" layer="95"/>
+<attribute name="VALUE" x="48.26" y="48.26" size="1.778" layer="96"/>
+</instance>
+<instance part="X" gate="-1" x="63.5" y="33.02" smashed="yes" rot="R90">
+<attribute name="NAME" x="62.611" y="33.02" size="1.778" layer="95" rot="R270"/>
+</instance>
+<instance part="X" gate="-2" x="68.58" y="33.02" smashed="yes" rot="R90">
+<attribute name="VALUE" x="72.263" y="30.48" size="1.778" layer="96" rot="R90"/>
+<attribute name="NAME" x="67.691" y="33.02" size="1.778" layer="95" rot="R270"/>
+</instance>
+<instance part="J1" gate="G$1" x="22.86" y="40.64" smashed="yes" rot="R180">
+<attribute name="NAME" x="25.4" y="33.02" size="1.778" layer="95" rot="R180"/>
+<attribute name="VALUE" x="25.4" y="51.308" size="1.778" layer="96" rot="R180"/>
+</instance>
+<instance part="R1" gate="G$1" x="33.02" y="35.56" smashed="yes" rot="R90">
+<attribute name="NAME" x="31.5214" y="31.75" size="1.778" layer="95" rot="R90"/>
+<attribute name="VALUE" x="36.322" y="31.75" size="1.778" layer="96" rot="R90"/>
+</instance>
+<instance part="U$3" gate="G$1" x="116.84" y="43.18" smashed="yes"/>
+<instance part="BZR" gate="G$1" x="48.26" y="83.82" smashed="yes">
+<attribute name="NAME" x="41.91" y="89.535" size="1.778" layer="95"/>
+<attribute name="VALUE" x="41.91" y="78.74" size="1.778" layer="96"/>
+</instance>
+<instance part="RELAY" gate="1" x="15.24" y="73.66" smashed="yes">
+<attribute name="VALUE" x="13.97" y="63.5" size="1.778" layer="96"/>
+<attribute name="NAME" x="13.97" y="79.502" size="1.778" layer="95"/>
+</instance>
+<instance part="LCD" gate="1" x="116.84" y="25.4" smashed="yes" rot="R180">
+<attribute name="VALUE" x="118.11" y="35.56" size="1.778" layer="96" rot="R180"/>
+<attribute name="NAME" x="118.11" y="19.558" size="1.778" layer="95" rot="R180"/>
+</instance>
 </instances>
 <busses>
@@
 <wire x1="68.58" y1="66.04" x2="73.66" y2="66.04" width="0.1524" layer="91"/>
 <wire x1="73.66" y1="66.04" x2="73.66" y2="73.66" width="0.1524" layer="91"/>
-<pinref part="U$3" gate="G$1" pin="LV_TXI_1"/>
+<pinref part="U$3" gate="G$1" pin="LV1"/>
 <wire x1="73.66" y1="73.66" x2="86.36" y2="73.66" width="0.1524" layer="91"/>
 </segment>
@@
 <wire x1="68.58" y1="63.5" x2="76.2" y2="63.5" width="0.1524" layer="91"/>
 <wire x1="76.2" y1="63.5" x2="76.2" y2="71.12" width="0.1524" layer="91"/>
-<pinref part="U$3" gate="G$1" pin="LV_RXO_1"/>
+<pinref part="U$3" gate="G$1" pin="LV2"/>
 <wire x1="76.2" y1="71.12" x2="86.36" y2="71.12" width="0.1524" layer="91"/>
 </segment>
@@
 <wire x1="104.14" y1="53.34" x2="139.7" y2="53.34" width="0.1524" layer="91"/>
 <wire x1="139.7" y1="53.34" x2="139.7" y2="73.66" width="0.1524" layer="91"/>
-<pinref part="U$3" gate="G$1" pin="HV_TXO_1"/>
+<pinref part="U$3" gate="G$1" pin="HV1"/>
 <wire x1="139.7" y1="73.66" x2="124.46" y2="73.66" width="0.1524" layer="91"/>
 <pinref part="LCD" gate="1" pin="4"/>
@@
 <wire x1="101.6" y1="50.8" x2="137.16" y2="50.8" width="0.1524" layer="91"/>
 <wire x1="137.16" y1="50.8" x2="137.16" y2="71.12" width="0.1524" layer="91"/>
-<pinref part="U$3" gate="G$1" pin="HV_RXI_1"/>
+<pinref part="U$3" gate="G$1" pin="HV2"/>
 <wire x1="137.16" y1="71.12" x2="124.46" y2="71.12" width="0.1524" layer="91"/>
 <pinref part="LCD" gate="1" pin="3"/>
